File: 003_GBungE_mk4_sch.kicad_sch (KiCad schematic)
At the start: 9 parts, among them K1 Relay Pre charge, K2 Relay AIR1, K3 timer relay, K4 Relay AIR2, M1 motor, SW1 LV_kill_SW, SW2 LV_Master_SW

Commit message: hen
Parts:
- added M2, M3: Fan, symbol Motor:Fan
- added M4: water_pump, symbol Motor:Fan
- added M5: accel, symbol Motor:Motor_Servo
- added SW3: HV_kill_SW, symbol Switch:SW_SPST
- added SW4: HV_Master_SW, symbol Switch:SW_SPST
- added SW5: FAN_SW, symbol Switch:SW_SPST
- added SW7: SW_SPDT, symbol Switch:SW_SPDT
Connections:
- net LV_battery/LV+: no longer SW1.1 (A)
- net at SW1.2 (B): no longer SW2.1 (A)
- new net motor controller/ACC+: M5.2 (+)
- new net motor controller/ACC-: M5.3 (-)
- new net motor controller/ACC_out: M5.1 (PWM)
- new net motor controller/FNR-: SW7.2 (B)
- new net motor controller/FNR_F: SW7.3 (C)
- new net motor controller/FNR_R: SW7.1 (A)
Other:
- added sheet LV_battery2 (titled2.kicad_sch)
- sheet motor controller ports: added ACC+, ACC-, ACC_out, FNR-, FNR_F, FNR_R; removed none
- note added: "전후진"
- moved on the sheet: C1, K1, K2, K3, K4, M1, R1, SW1, SW2
