File: titled.kicad_sch (KiCad schematic)
At the start: 1 part, among them J1 sevcon gen4 main

Commit message: hen
Connections:
- no-connect marks 3 -> 7
Changed lines of the file:
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@@
 	(paper "A4")
 	(no_connect
+		(at 104.14 66.04)
+	)
+	(no_connect
 		(at 81.28 110.49)
 	)
 	(no_connect
+		(at 104.14 60.96)
+	)
+	(no_connect
 		(at 81.28 102.87)
 	)
 	(no_connect
+		(at 83.82 66.04)
+	)
+	(no_connect
+		(at 83.82 63.5)
+	)
+	(no_connect
 		(at 81.28 107.95)
 	)
+	(wire
+		(pts
+			(xy 73.66 86.36) (xy 81.28 86.36)
+		)
+		(stroke
+			(width 0)
+			(type default)
+		)
+	)
+	(wire
+		(pts
+			(xy 73.66 91.44) (xy 81.28 91.44)
+		)
+		(stroke
+			(width 0)
+			(type default)
+		)
+	)
+	(wire
+		(pts
+			(xy 73.66 88.9) (xy 81.28 88.9)
+		)
+		(stroke
+			(width 0)
+			(type default)
+		)
+	)
+	(wire
+		(pts
+			(xy 73.66 81.28) (xy 81.28 81.28)
+		)
+		(stroke
+			(width 0)
+			(type default)
+		)
+	)
+	(wire
+		(pts
+			(xy 73.66 83.82) (xy 81.28 83.82)
+		)
+		(stroke
+			(width 0)
+			(type default)
+		)
+	)
+	(label "bat-"
+		(at 104.14 58.42 0)
+		(effects
+			(font
+				(size 1.27 1.27)
+				(thickness 0.254)
+				(bold yes)
+			)
+			(justify left bottom)
+		)
+	)
+	(label "bat-"
+		(at 76.2 88.9 0)
+		(effects
+			(font
+				(size 1.27 1.27)
+				(thickness 0.254)
+				(bold yes)
+			)
+			(justify left bottom)
+		)
+	)
+	(label "bat-"
+		(at 83.82 58.42 0)
+		(effects
+			(font
+				(size 1.27 1.27)
+				(thickness 0.254)
+				(bold yes)
+			)
+			(justify left bottom)
+		)
+	)
+	(hierarchical_label "ACC_out"
+		(shape input)
+		(at 104.14 66.04 180)
+		(effects
+			(font
+				(size 1.27 1.27)
+			)
+			(justify right)
+		)
+	)
 	(hierarchical_label "+"
 		(shape input)
-		(at 81.28 83.82 180)
+		(at 73.66 83.82 180)
 		(effects
 			(font
@@
 	(hierarchical_label "U"
 		(shape input)
-		(at 81.28 81.28 180)
+		(at 73.66 81.28 180)
+		(effects
+			(font
+				(size 1.27 1.27)
+			)
+			(justify right)
+		)
+	)
+	(hierarchical_label "ACC-"
+		(shape input)
+		(at 104.14 58.42 180)
 		(effects
 			(font
@@
 	(hierarchical_label "-"
 		(shape input)
-		(at 81.28 88.9 180)
+		(at 73.66 88.9 180)
 		(effects
 			(font
@@
 	(hierarchical_label "W"
 		(shape input)
-		(at 81.28 91.44 180)
+		(at 73.66 91.44 180)
+		(effects
+			(font
+				(size 1.27 1.27)
+			)
+			(justify right)
+		)
+	)
+	(hierarchical_label "FNR_R"
+		(shape input)
+		(at 83.82 66.04 180)
+		(effects
+			(font
+				(size 1.27 1.27)
+			)
+			(justify right)
+		)
+	)
+	(hierarchical_label "FNR-"
+		(shape input)
+		(at 83.82 58.42 180)
 		(effects
 			(font
@@
 		)
 	)
+	(hierarchical_label "ACC+"
+		(shape input)
+		(at 104.14 60.96 180)
+		(effects
+			(font
+				(size 1.27 1.27)
+			)
+			(justify right)
+		)
+	)
+	(hierarchical_label "FNR_F"
+		(shape input)
+		(at 83.82 63.5 180)
+		(effects
+			(font
+				(size 1.27 1.27)
+			)
+			(justify right)
+		)
+	)
 	(hierarchical_label "V"
 		(shape input)
-		(at 81.28 86.36 180)
-		(effects
-			(font
+		(at 73.66 86.36 180)
+		(effects
+			(font
